File: pat80-computer/hardware/schematics/pat80/pat80.kicad_pcb (KiCad board)
At the start: 2 copper layers, 44 parts, among them J1 panel_btn_brk, J2 Power input, J3 panel_led_halt, J4 panel_btn_rst, J5 nmi, SW1 SW_Push, SW2 Break, U1 Z80CPU, U10 74HC32, U11 74HC04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

Commit message: WIP mainboard routing
Routing:
- net /D7: track 34.4 -> 162.5 mm, vias 0 -> 4
- net /D1: track 70.4 -> 184.6 mm, vias 0 -> 2
- net /D6: track 34.4 -> 147.9 mm, vias 0 -> 2
- net /D5: track 34.4 -> 145.4 mm, vias 0 -> 2
- net /D4: track 34.4 -> 145.4 mm, vias 0 -> 2
- net /D3: track 34.4 -> 137.8 mm, vias 0 -> 2
- net /D2: track 75.2 -> 159.5 mm, vias 2 -> 4
- net Net-(U1-Pad6): track 0.00 -> 68.6 mm, vias 0 -> 2
- net VCC: track 34.2 -> 84.9 mm
- net /A15: track 0.00 -> 44.8 mm, vias 0 -> 2
- net Net-(U10-Pad1): track 0.00 -> 34.0 mm
