File: pat80-io-devices/keyboard/hardware/keyboard/keyboard.kicad_pcb (KiCad board)
At the start: 2 copper layers, 273.1 x 144.8 mm, 123 parts, among them J3 Keyboard connector, SW1 1, SW10 3, SW11 E, SW12 D, SW13 C, SW14 V, SW15 F, SW16 R, SW17 4, SW18 5, SW19 T, SW2 Q, SW20 G, SW21 B, SW22 N, SW23 H, SW24 Y, SW25 6, SW26 7, SW27 U, SW28 J, SW29 M, SW3 A, SW30 ', SW31 K, SW32 I, SW33 8, SW34 9, SW35 O, SW36 L, SW37 P, SW38 [, SW39 ], SW4 Z, SW40 0, SW41 BACKSPACE, SW42 TILDE, SW43 TAB, SW44 ,, SW45 ., SW46 SPACE, SW47 /, SW48 ;, SW49 LSHIFT, SW5 X, SW50 CTRL, SW51 RSHIFT, SW52 RETURN, SW53 PATO, SW54 CAPSLK, SW6 S, SW7 W, SW8 2

Commit message: Refinement
Routing:
- net Net-(D9-Pad2): track 16.9 -> 14.9 mm
Changed lines of the file:
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@@
     (thickness 1.6)
     (drawings 8)
-    (tracks 761)
+    (tracks 762)
     (zones 0)
     (modules 123)
@@
   (page A4)
   (layers
-    (0 F.Cu signal)
+    (0 F.Cu signal hide)
     (31 B.Cu signal)
-    (32 B.Adhes user)
-    (33 F.Adhes user)
-    (34 B.Paste user)
-    (35 F.Paste user)
-    (36 B.SilkS user)
-    (37 F.SilkS user)
-    (38 B.Mask user)
-    (39 F.Mask user)
-    (40 Dwgs.User user)
-    (41 Cmts.User user)
-    (42 Eco1.User user)
-    (43 Eco2.User user)
+    (32 B.Adhes user hide)
+    (33 F.Adhes user hide)
+    (34 B.Paste user hide)
+    (35 F.Paste user hide)
+    (36 B.SilkS user hide)
+    (37 F.SilkS user hide)
+    (38 B.Mask user hide)
+    (39 F.Mask user hide)
+    (40 Dwgs.User user hide)
+    (41 Cmts.User user hide)
+    (42 Eco1.User user hide)
+    (43 Eco2.User user hide)
     (44 Edge.Cuts user)
-    (45 Margin user)
-    (46 B.CrtYd user)
-    (47 F.CrtYd user)
-    (48 B.Fab user)
-    (49 F.Fab user)
+    (45 Margin user hide)
+    (46 B.CrtYd user hide)
+    (47 F.CrtYd user hide)
+    (48 B.Fab user hide)
+    (49 F.Fab user hide)
   )
   (setup
@@
   (segment (start 34.29 107.95) (end 34.29 105.0798) (width 0.5) (layer B.Cu) (net 12))
   (segment (start 26.035 122.428) (end 26.416 122.809) (width 0.5) (layer B.Cu) (net 13))
-  (segment (start 26.035 106.045) (end 26.035 122.428) (width 0.5) (layer B.Cu) (net 13))
+  (segment (start 26.416 108.966) (end 26.035 108.585) (width 0.5) (layer B.Cu) (net 13))
+  (segment (start 26.416 122.809) (end 26.416 108.966) (width 0.5) (layer B.Cu) (net 13))
   (segment (start 89.535 56.769) (end 89.408 56.896) (width 0.5) (layer B.Cu) (net 14))
   (segment (start 89.535 53.34) (end 89.535 56.769) (width 0.5) (layer B.Cu) (net 14))
